File: Eagle/Sidney 2019 boards/Motor board.sch (EAGLE design)
At the start: 26 parts, among them IC1 LM2596S, J1 TWIG_2.0, J2 TWIG_2.0, J3 TWIG_2.0, J4 TWIG_2.0

Commit message: supply improvements in motor board
Parts:
- added IC2: LM2940CS-5.0_NOPB, LM2940CS-5.0_NOPB:LM2940CS-5.0_NOPB
Connections:
- removed net ALIM_ELE: C2.+, C4.1, IC1.VIN
- net 5.7V-DIRAMAZIONE2: now also IC2.IN
- net GND: now also IC2.GND, IC2.GND_(TAB)
- net VCC: now also C2.+, C4.1, IC1.VIN
Other:
- moved on the sheet: C2, C4, C5, C6, D1, D2, IC1, J1, J2, J3, J4, LED2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

Commit message: general improvements to the boards
Parts:
- removed C10, C11: 12065D106KAT2A, 12065D106KAT2A:12065D106KAT2A
- removed TP1: TPTP13SQ, testpad:TPTP13SQ
- removed U$3: (no value), inductor-coilcraft:MSS1260
- added C1: (no value), rcl:C-EUC1206
- added C3, C7: (no value), cap-pan40:C-PR-SMD-SV-E/F
- added C8: (no value), eagle-ltspice:CC1206
- added L1: 47/470uH (?), inductor-coilcraft:MSS1260
- added SUPPLY_CON: (no value), con-molex-micro-fit-3_0:HEADER_POS4_43045-0412
- C2: device cap-pan40:C-PR-SMD-SV-E/F -> rcl:C-EUC1206
Connections:
- removed net N$8: LED2.K, R3.2
- new net +5V/S: C8.1, IC2.OUT
- new net N$3: LED2.A, R3.1
- net +5V: now also R3.2; no longer LED2.A, TP1.TP
- net 5.7V-DIRAMAZIONE2: now also C7.+, L1.P$1; no longer U$3.P$1
- net GND: now also C1.2, C2.2, C3.-, C7.-, C8.2, LED2.K; no longer C10.2, C11.2, C2.-, R3.1
- net N$6: now also L1.P$2; no longer U$3.P$2
- net VCC: now also C1.1, C3.+; no longer C10.1, C2.+
- net VMOT: now also C2.1; no longer C11.1
Other:
- note added: "SUPPLY"
- note added: "SUPPLY_SW"
- moved on the sheet: C4, C5, C6, D1, D2, IC1, IC2, J1, J2, J3, J4, LED2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

Commit message: finished motor drivers (schematic)
Parts:
- removed J1, J2, J3, J4: TWIG_2.0, CONNECTER:TWIG_2.0
- removed MOTOR_DRIVER_A, MOTOR_DRIVER_B, MOTOR_DRIVER_C, MOTOR_DRIVER_D: VNH5019, DRIVER POLOLU:VNH5019
- added MOTOR_DRIVER_1, MOTOR_DRIVER_2, MOTOR_DRIVER_3, MOTOR_DRIVER_4: VNH5019, DRIVER POLOLU:VNH5019
- added MOT_1, MOT_2, MOT_3, MOT_4: MST2V, con-phoenix-508:MST2V
- added S1, S2, S3, S4: TWIG_2.0, CONNECTER:TWIG_2.0
- added SIGN_CON: (no value), con-harting-v-edit:20V
- SUPPLY_CON: value (none) -> 39-28-1043; device con-molex-micro-fit-3_0:HEADER_POS4_43045-0412 -> 39-28-1043:39-28-1043
Connections:
- new net M1_A: MOTOR_DRIVER_1.A, MOT_1-1.1
- new net M1_B: MOTOR_DRIVER_1.B, MOT_1-2.1
- new net M1_INA: MOTOR_DRIVER_1.IN_A, SIGN_CON.8
- new net M1_INB: MOTOR_DRIVER_1.IN_B, SIGN_CON.10
- new net M1_PWM: MOTOR_DRIVER_1.PWM, SIGN_CON.2
- new net M2_A: MOTOR_DRIVER_2.A, MOT_2-1.1
- new net M2_B: MOTOR_DRIVER_2.B, MOT_2-2.1
- new net M2_INA: MOTOR_DRIVER_2.IN_A, SIGN_CON.12
- new net M2_INB: MOTOR_DRIVER_2.IN_B, SIGN_CON.14
- new net M2_PWM: MOTOR_DRIVER_2.PWM, SIGN_CON.4
- new net M3_A: MOTOR_DRIVER_3.A, MOT_3-1.1
- new net M3_B: MOTOR_DRIVER_3.B, MOT_3-2.1
- new net M3_INA: MOTOR_DRIVER_3.IN_A, SIGN_CON.16
- new net M3_INB: MOTOR_DRIVER_3.IN_B, SIGN_CON.18
- new net M3_PWM: MOTOR_DRIVER_3.PWM, SIGN_CON.6
- new net M4_A: MOTOR_DRIVER_4.A, MOT_4-1.1
- new net M4_B: MOTOR_DRIVER_4.B, MOT_4-2.1
- new net M4_INA: MOTOR_DRIVER_4.IN_A, SIGN_CON.3
- new net M4_INB: MOTOR_DRIVER_4.IN_B, SIGN_CON.5
- new net M4_PWM: MOTOR_DRIVER_4.PWM, SIGN_CON.1
- new net S1_DOWN: S1.2, SIGN_CON.19
- new net S1_UP: S1.1, SIGN_CON.20
- new net S2_DOWN: S2.2, SIGN_CON.15
- new net S2_UP: S2.1, SIGN_CON.17
- new net S3_DOWN: S3.2, SIGN_CON.11
- new net S3_UP: S3.1, SIGN_CON.13
- new net S4_DOWN: S4.2, SIGN_CON.7
- new net S4_UP: S4.1, SIGN_CON.9
- net +5V: now also SUPPLY_CON.3
- net +5V/S: now also MOTOR_DRIVER_1.+5V, MOTOR_DRIVER_2.+5V, MOTOR_DRIVER_3.+5V, MOTOR_DRIVER_4.+5V, S1.3, S2.3, S3.3, S4.3, SUPPLY_CON.2
- net GND: now also MOTOR_DRIVER_1.GND, MOTOR_DRIVER_2.GND, MOTOR_DRIVER_3.GND, MOTOR_DRIVER_4.GND, S1.4, S2.4, S3.4, S4.4, SUPPLY_CON.1, SUPPLY_CON.4
- net VMOT: now also MOTOR_DRIVER_1.+12V, MOTOR_DRIVER_2.+12V, MOTOR_DRIVER_3.+12V, MOTOR_DRIVER_4.+12V
Other:
- note added: "LINE_CONS"
- note added: "MOTOR_DRIVERS"
- note added: "MOT_CONS"
- moved on the sheet: SUPPLY_CON
