File: Eagle/Sidney 2019 boards/Line sensors.sch (EAGLE design)
At the start: 19 parts

Commit message: Almost completed components lists
Parts:
- removed C5: 100n, resistor:R-EU_M0805
- removed D5: (no value), Wurth_Elektronik_Optoelectronics_rev15b:WL-SMTW-150141AS73100-A
- removed LED5: (no value), SparkFun:LED3MM
- removed R14: 10k, resistor:R-EU_M0805
- added C1: 100n, resistor:R-EU_M0805
- added D1: (no value), Wurth_Elektronik_Optoelectronics_rev15b:WL-SMTW-150141AS73100-A
- added LED1: (no value), SparkFun:LED3MM
- added R1: 330, resistor:R-EU_M0805
- R5: value 330 -> 10k
- renumbered C7 to C4, D7 to D4, LED7 to LED4, R13 to R4, R9 to R3
Connections:
- removed net N$4 (its old number): D3.A, R5.1
- new net N$3: D1.A, R1.1
- net 5V: now also C1.2, LED1.A, R1.2; no longer C5.2, LED5.A, R5.2
- net GND: now also C1.1, D1.K, R5.1; no longer C5.1, D5.K, R14.1
- net N$13: now also D3.A; no longer D5.A
- net SIG1: now also LED1.C, R5.2; no longer LED3.C, R6.2
- net SIG2: now also LED3.C, R6.2; no longer LED5.C, R14.2
Other:
- moved on the sheet: C2, C3, D2, D3, LED2, LED3, R2, R5, R6
